File: Badge Balam/Badge Balam.kicad_pcb (KiCad board)
At the start: 2 copper layers, 46.3 x 63.1 mm, 6 parts

Commit message: cambios
Parts:
- removed BT1: BAT-HLD-001, Battery:BatteryHolder_Keystone_3002_1x2032
- removed the REF** at (192.0, 70.8)
- added REF**: SW_EG1218, EG1218:SW_EG1218, B.Cu at (166.1, 84.6)
- added REF**: BatteryHolder_Keystone_3002_1x2032, Battery:BatteryHolder_Keystone_3002_1x2032, B.Cu at (150.2, 72.0)
Connections:
- net Net-(D1-A) renamed /diode_flag
Routing:
- net GNDREF: track 0.00 -> 47.4 mm
- net /diode_flag: track 0.00 -> 35.5 mm
- added copper zone on F.Cu, net (none)
- added copper zone on B.Cu, net +3V0
